Commit message: 1.update MotionCommands msg 2.add hardware_neck pkg

File: share/description/model/urdf/elf2-trunk/urdf/elf2_trunk_dof12.urdf (robot description, URDF)
Before this commit: robot elf2, 28 links, 27 joints
Links:
- removed link d435i
- removed link mid360
Joints:
- removed joint d435i_joint
- removed joint mid360_joint

File: share/description/model/urdf/elf2-trunk/urdf/elf2_trunk_dof25.urdf (robot description, URDF)
Before this commit: robot elf2, 28 links, 27 joints
Links:
- removed link d435i
- removed link mid360
Joints:
- removed joint d435i_joint
- removed joint mid360_joint
